File: KiCAD/Cartridge_800xl_4/Cartridge_800xl_2.kicad_pcb (KiCad board)
At the start: 4 copper layers, 64 x 80.2 mm, 21 parts, among them SW1 Reset, U1 27C512, U2 74HC165, U3 74HC595, U4 GAL16V8, U5 TXS0108EPW, U6 mini_esp32

Commit message: pcb update
Connections:
- U5 pad 3: iIO1 -> IO1L
Routing:
- net iIO1: track 25.6 -> 0.00 mm, vias 1 -> 0
- net IO1L: track 0.00 -> 25.6 mm, vias 0 -> 1

Commit message: servercode
Routing:
- net GND: track 11.6 -> 0.21 mm, vias 11 -> 12
- net sclk_2: track 19.5 -> 15.6 mm, vias 0 -> 1
- net sclk_1L: track 15.3 -> 14.0 mm

Commit message: pcb update
Parts:
- moved Z1 2.43 mm to (133.7, 138.8)
Other:
- board size 64 x 80.2 mm -> 64 x 82.6 mm
Changed lines of the file:
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@@
 	(footprint "Barts:Atari_bus"
 		(layer "F.Cu")
-		(at 133.7745 136.358)
+		(at 133.671352 138.782)
 		(property "Reference" "Z1"
 			(at 0 5.08 180)
@@
 	)
 	(gr_line
-		(start 132.245148 140.3875)
-		(end 132.245148 123.7625)
+		(start 131.953 142.8115)
+		(end 131.953 123.7615)
 		(stroke
 			(width 0.1)
@@
 	)
 	(gr_line
-		(start 119.695148 123.7625)
-		(end 132.245148 123.7625)
+		(start 171.0055 142.8115)
+		(end 171.0055 123.8125)
 		(stroke
 			(width 0.1)
-			(type solid)
+			(type default)
 		)
 		(layer "Edge.Cuts")
 	)
 	(gr_line
-		(start 183.570148 60.1625)
-		(end 119.670148 60.1625)
+		(start 119.695148 123.7625)
+		(end 131.953 123.7615)
 		(stroke
 			(width 0.1)
@@
 	)
 	(gr_line
-		(start 119.695148 123.7625)
+		(start 183.570148 60.1625)
 		(end 119.670148 60.1625)
 		(stroke
@@
 	)
 	(gr_line
-		(start 183.670148 123.7875)
-		(end 171.055148 123.8125)
+		(start 119.695148 123.7625)
+		(end 119.670148 60.1625)
 		(stroke
 			(width 0.1)
@@
 	)
 	(gr_line
-		(start 171.045148 140.3875)
-		(end 171.055148 123.8125)
+		(start 183.670148 123.7875)
+		(end 171.0055 123.8125)
 		(stroke
 			(width 0.1)
@@
 	)
 	(gr_line
-		(start 171.045148 140.3875)
-		(end 132.245148 140.3875)
+		(start 171.0055 142.8115)
+		(end 131.953 142.8115)
 		(stroke
 			(width 0.1)
@@
 		(layer "User.1")
 		(pts
-			(xy 183.570148 60.2125) (xy 183.645148 140.4625)
+			(xy 183.570148 60.2125) (xy 183.5785 142.8115)
 		)
 		(height -13.374858)
@@
 			(keep_text_aligned yes)
 		)
-		(gr_text "80.2500 mm"
-			(at 198.132499 100.323925 270.0535474)
+		(gr_text "82.5990 mm"
+			(at 198.099182 101.510532 270.0057935)
 			(layer "User.1")
 			(effects
@@
 		(layer "User.1")
 		(pts
-			(xy 132.245148 140.3875) (xy 171.045148 140.3875)
+			(xy 131.953 142.8115) (xy 171.0055 142.8115)
 		)
 		(height 4.45)
@@
 			(keep_text_aligned yes)
 		)
-		(gr_text "38.8000 mm"
-			(at 151.645148 143.6875 0)
+		(gr_text "39.0525 mm"
+			(at 151.47925 146.1115 0)
 			(layer "User.1")
 			(effects

Commit message: small changes
Routing:
- net A3: track 15.3 -> 21.7 mm
- net A5: track 19.6 -> 22.8 mm
- net A1: track 68.3 -> 71.2 mm
- net D3: track 101.8 -> 104.7 mm
- net ~{S5}: track 59.1 -> 61.9 mm
- net A10: track 53.9 -> 56.6 mm
- net D5: track 80.1 -> 82.4 mm
- net A11: track 46.3 -> 48.6 mm
- net A8: track 36.8 -> 38.8 mm
- net R/~{W}: track 26.4 -> 25.8 mm

Commit message: pcb update
Parts:
- C1, C3, C4, C5, C6, C7, C8, C9: value 100n -> 100nF
- D1: value LED -> LED red
- R2: value 10k -> 10kΩ
- moved C6 2.10 mm to (137.4, 118.2)
- moved Z1 0.21 mm to (133.9, 138.7)
Routing:
- net +5V: track 201.6 -> 202.3 mm
- net A3: track 21.7 -> 21.0 mm
Other:
- board size 64 x 82.6 mm -> 63.9 x 82.6 mm
